File: Accumulate_functional.kicad_sch (KiCad schematic)
At the start: 0 parts

Commit message: VER1.0: добавил два листа с арматурами
Other:
- added sheet Accum (Accum.kicad_sch)
- added sheet ECG (ECG.kicad_sch)
Changed lines of the file:
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@@
+		)
+	)
+	(sheet
+		(at 858.52 0)
+		(size 59.69 44.45)
+		(exclude_from_sim no)
+		(in_bom yes)
+		(on_board yes)
+		(dnp no)
+		(fields_autoplaced yes)
+		(stroke
+			(width 0.1524)
+			(type solid)
+		)
+		(fill
+			(color 0 0 0 0)
+		)
+		(property "Sheetname" "ECG"
+			(at 858.52 -0.7116 0)
+			(show_name no)
+			(do_not_autoplace no)
+			(effects
+				(font
+					(size 1.27 1.27)
+				)
+				(justify left bottom)
+			)
+		)
+		(property "Sheetfile" "ECG.kicad_sch"
+			(at 858.52 45.0346 0)
+			(show_name no)
+			(do_not_autoplace no)
+			(effects
+				(font
+					(size 1.27 1.27)
+				)
+				(justify left top)
+			)
+		)
+		(instances
+			(project "Accumulate_functional"
+				(path "/99fca793-e79a-435a-82d3-c27bbf906660"
+					(page "2")
+				)
+			)
+		)
+	)
+	(sheet
+		(at 858.52 52.07)
+		(size 59.69 44.45)
+		(exclude_from_sim no)
+		(in_bom yes)
+		(on_board yes)
+		(dnp no)
+		(fields_autoplaced yes)
+		(stroke
+			(width 0.1524)
+			(type solid)
+		)
+		(fill
+			(color 0 0 0 0)
+		)
+		(property "Sheetname" "Accum"
+			(at 858.52 51.3584 0)
+			(show_name no)
+			(do_not_autoplace no)
+			(effects
+				(font
+					(size 1.27 1.27)
+				)
+				(justify left bottom)
+			)
+		)
+		(property "Sheetfile" "Accum.kicad_sch"
+			(at 858.52 97.1046 0)
+			(show_name no)
+			(do_not_autoplace no)
+			(effects
+				(font
+					(size 1.27 1.27)
+				)
+				(justify left top)
+			)
+		)
+		(instances
+			(project "Accumulate_functional"
+				(path "/99fca793-e79a-435a-82d3-c27bbf906660"
+					(page "3")
+				)
+			)
 		)
 	)

Commit message: VER1.0: добавил зоны помещений
Other:
- note added: "Наружний шкаф"
- note added: "Помещение 1"
- note added: "Помещение 2"
Changed lines of the file:
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@@
 	(generator_version "10.0")
 	(paper "A1")
+	(rectangle
+		(start 124.46 447.04)
+		(end 264.16 546.1)
+		(stroke
+			(width 0.508)
+			(type dash)
+			(color 0 0 0 1)
+		)
+		(fill
+			(type color)
+			(color 255 153 0 0.2705882353)
+		)
+	)
+	(rectangle
+		(start 124.46 284.48)
+		(end 264.16 444.5)
+		(stroke
+			(width 0.508)
+			(type dash)
+			(color 0 0 0 1)
+		)
+		(fill
+			(type color)
+			(color 255 0 0 0.2588235294)
+		)
+	)
 	(text "Питание 24В"
 		(exclude_from_sim no)
@@
 		)
 	)
+	(text "Помещение 1"
+		(exclude_from_sim no)
+		(at 452.882 412.496 0)
+		(effects
+			(font
+				(face "Calibri")
+				(size 5.08 5.08)
+				(bold yes)
+				(italic yes)
+				(color 0 0 0 1)
+			)
+		)
+	)
+	(text "Помещение 2"
+		(exclude_from_sim no)
+		(at 257.556 367.792 90)
+		(effects
+			(font
+				(face "Calibri")
+				(size 5.08 5.08)
+				(bold yes)
+				(italic yes)
+				(color 0 0 0 1)
+			)
+		)
+	)
 	(text "Напряжение переменное AC (сеть)"
 		(exclude_from_sim no)
@@
 			)
 			(justify left)
+		)
+	)
+	(text "Наружний шкаф"
+		(exclude_from_sim no)
+		(at 192.278 535.94 0)
+		(effects
+			(font
+				(face "Calibri")
+				(size 5.08 5.08)
+				(bold yes)
+				(italic yes)
+				(color 0 0 0 1)
+			)
 		)
 	)
@@
 	(polyline
 		(pts
+			(xy 274.32 444.5) (xy 274.32 281.94)
+		)
+		(stroke
+			(width 0.508)
+			(type dash)
+			(color 0 0 0 1)
+		)
+	)
+	(polyline
+		(pts
 			(xy 614.68 170.18) (xy 662.94 170.18)
 		)
@@
 	(polyline
 		(pts
+			(xy 124.46 281.94) (xy 274.32 281.94)
+		)
+		(stroke
+			(width 0.508)
+			(type dash)
+			(color 0 0 0 1)
+		)
+	)
+	(polyline
+		(pts
 			(xy 195.58 360.68) (xy 195.58 370.84)
 		)
@@
 	(polyline
 		(pts
+			(xy 523.24 274.32) (xy 647.7 274.32)
+		)
+		(stroke
+			(width 0.508)
+			(type dash)
+			(color 0 0 0 1)
+		)
+	)
+	(polyline
+		(pts
+			(xy 124.46 281.94) (xy 124.46 25.4)
+		)
+		(stroke
+			(width 0.508)
+			(type dash)
+			(color 0 0 0 1)
+		)
+	)
+	(polyline
+		(pts
 			(xy 449.58 241.3) (xy 576.58 241.3)
 		)
@@
 	(polyline
 		(pts
+			(xy 124.46 25.4) (xy 523.24 25.4)
+		)
+		(stroke
+			(width 0.508)
+			(type dash)
+			(color 0 0 0 1)
+		)
+	)
+	(polyline
+		(pts
 			(xy 322.58 360.68) (xy 322.58 406.4)
 		)
@@
 		)
 	)
+	(polyline
+		(pts
+			(xy 647.7 444.5) (xy 274.32 444.5)
+		)
+		(stroke
+			(width 0.508)
+			(type dash)
+			(color 0 0 0 1)
+		)
+	)
 	(wire
 		(pts
@@
 	(polyline
 		(pts
+			(xy 647.7 274.32) (xy 647.7 444.5)
+		)
+		(stroke
+			(width 0.508)
+			(type dash)
+			(color 0 0 0 1)
+		)
+	)
+	(polyline
+		(pts
 			(xy 45.72 530.86) (xy 60.96 530.86)
 		)
@@
 		)
 	)
+	(polyline
+		(pts
+			(xy 523.24 25.4) (xy 523.24 274.32)
+		)
+		(stroke
+			(width 0.508)
+			(type dash)
+			(color 0 0 0 1)
+		)
+	)
