File: Accumulate_functional.kicad_sch (KiCad schematic)
At the start: 0 parts

Commit message: refactor for new ver
Other:
- note added: "CAN сеть (КИС-В)"
- note added: "HDMI-кабель"
- note added: "Высокое напряжение постоянное DC 100мм2 (например, EV-Cable или ППГнг(А)-HF)"
- note added: "Напряжение переменное AC (сеть) 4х 150 кв.мм(например, ППГнг(А)-HF)"
- note added: "Питание 24В 2 x 1,5кв.мм (например, ПВС)"
- note added: "Управление 24В 2 х 1,5 кв.мм (например МКЭШ 1,5)"
- note added: "трехфазный провод с нейтралью 4х10кв.мм (например, КГтп-ХЛ 4х10)"
- note removed: "CAN сеть"
- note removed: "HDMI"
- note removed: "Высокое напряжение постоянное DC"
- note removed: "Напряжение переменное AC (сеть)"
- note removed: "Питание 24В"
- note removed: "Управление 24В"
Changed lines of the file:
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@@
 		)
 	)
-	(text "Питание 24В"
+	(text "Питание 24В 2 x 1,5кв.мм (например, ПВС)"
 		(exclude_from_sim no)
 		(at 63.5 546.1 0)
@@
 		)
 	)
-	(text "CAN сеть"
+	(text "трехфазный провод с нейтралью 4х10кв.мм (например, КГтп-ХЛ 4х10)"
+		(exclude_from_sim no)
+		(at 63.754 562.61 0)
+		(effects
+			(font
+				(face "Calibri")
+				(size 2.54 2.54)
+				(thickness 0.254)
+				(bold yes)
+				(italic yes)
+				(color 0 0 0 1)
+			)
+			(justify left)
+		)
+	)
+	(text "CAN сеть (КИС-В)"
 		(exclude_from_sim no)
 		(at 63.5 541.02 0)
@@
 		)
 	)
-	(text "Напряжение переменное AC (сеть)"
+	(text "Напряжение переменное AC (сеть) 4х 150 кв.мм(например, ППГнг(А)-HF)"
 		(exclude_from_sim no)
 		(at 63.5 530.86 0)
@@
 		)
 	)
-	(text "HDMI"
+	(text "HDMI-кабель"
 		(exclude_from_sim no)
 		(at 63.5 556.26 0)
@@
 		)
 	)
-	(text "Высокое напряжение постоянное DC"
+	(text "Высокое напряжение постоянное DC 100мм2 (например, EV-Cable или ППГнг(А)-HF)"
 		(exclude_from_sim no)
 		(at 63.5 535.94 0)
@@
 		)
 	)
-	(text "Управление 24В"
+	(text "Управление 24В 2 х 1,5 кв.мм (например МКЭШ 1,5)"
 		(exclude_from_sim no)
 		(at 63.5 551.18 0)
@@
 		)
 	)
-	(text_box "ШКАФ ОТБОРА МОЩНОСТИ\nDC/DC\n"
+	(text_box "ШКАФ ОТБОРА МОЩНОСТИ\nAC/DC\n"
 		(exclude_from_sim no)
 		(at 601.98 144.78 0)
@@
 			(width 1.27)
 			(type default)
-			(color 194 0 194 1)
+			(color 120 100 50 1)
 		)
 	)
@@
 			(width 1.27)
 			(type default)
-			(color 194 0 194 1)
+			(color 120 100 50 1)
 		)
 	)
@@
 	(wire
 		(pts
-			(xy 646.43 215.9) (xy 646.43 252.73)
-		)
-		(stroke
-			(width 1.27)
-			(type default)
-			(color 194 0 194 1)
+			(xy 711.2 191.77) (xy 711.2 284.48)
+		)
+		(stroke
+			(width 1.27)
+			(type default)
+			(color 50 0 50 1)
 		)
 	)
@@
 	(wire
 		(pts
+			(xy 109.22 118.11) (xy 121.92 118.11)
+		)
+		(stroke
+			(width 1.27)
+			(type default)
+			(color 50 0 50 1)
+		)
+	)
+	(wire
+		(pts
 			(xy 458.47 59.69) (xy 648.97 59.69)
 		)
@@
 			(type solid)
 			(color 0 194 0 1)
+		)
+	)
+	(wire
+		(pts
+			(xy 109.22 284.48) (xy 711.2 284.48)
+		)
+		(stroke
+			(width 1.27)
+			(type default)
+			(color 50 0 50 1)
 		)
 	)
@@
 			(width 1.27)
 			(type default)
+			(color 120 100 50 1)
+		)
+	)
+	(wire
+		(pts
+			(xy 648.97 59.69) (xy 648.97 144.78)
+		)
+		(stroke
+			(width 1.27)
+			(type default)
+			(color 194 0 0 1)
+		)
+	)
+	(polyline
+		(pts
+			(xy 45.72 561.34) (xy 60.96 561.34)
+		)
+		(stroke
+			(width 1.27)
+			(type solid)
+			(color 120 100 50 1)
+		)
+	)
+	(polyline
+		(pts
+			(xy 236.22 120.65) (xy 261.62 120.65)
+		)
+		(stroke
+			(width 1.27)
+			(type solid)
+			(color 0 194 0 1)
+		)
+	)
+	(polyline
+		(pts
+			(xy 236.22 166.37) (xy 261.62 166.37)
+		)
+		(stroke
+			(width 1.27)
+			(type solid)
+			(color 0 194 0 1)
+		)
+	)
+	(polyline
+		(pts
+			(xy 483.87 175.26) (xy 497.84 175.26)
+		)
+		(stroke
+			(width 1.27)
+			(type solid)
+			(color 0 194 0 1)
+		)
+	)
+	(polyline
+		(pts
+			(xy 773.43 85.09) (xy 821.69 85.09)
+		)
+		(stroke
+			(width 2.54)
+			(type solid)
 			(color 194 0 194 1)
 		)
 	)
-	(wire
-		(pts
-			(xy 648.97 59.69) (xy 648.97 144.78)
-		)
-		(stroke
-			(width 1.27)
-			(type default)
-			(color 194 0 0 1)
-		)
-	)
-	(polyline
-		(pts
-			(xy 236.22 120.65) (xy 261.62 120.65)
-		)
-		(stroke
-			(width 1.27)
-			(type solid)
-			(color 0 194 0 1)
-		)
-	)
-	(polyline
-		(pts
-			(xy 236.22 166.37) (xy 261.62 166.37)
-		)
-		(stroke
-			(width 1.27)
-			(type solid)
-			(color 0 194 0 1)
-		)
-	)
-	(polyline
-		(pts
-			(xy 483.87 175.26) (xy 497.84 175.26)
-		)
-		(stroke
-			(width 1.27)
-			(type solid)
-			(color 0 194 0 1)
-		)
-	)
-	(polyline
-		(pts
-			(xy 773.43 85.09) (xy 821.69 85.09)
+	(polyline
+		(pts
+			(xy 433.07 217.17) (xy 433.07 227.33)
+		)
+		(stroke
+			(width 1.27)
+			(type solid)
+			(color 194 0 0 1)
+		)
+	)
+	(polyline
+		(pts
+			(xy 179.07 121.92) (xy 179.07 166.37)
+		)
+		(stroke
+			(width 1.27)
+			(type solid)
+			(color 0 194 0 1)
+		)
+	)
+	(wire
+		(pts
+			(xy 218.44 179.07) (xy 218.44 41.91)
+		)
+		(stroke
+			(width 1.27)
+			(type default)
+			(color 194 0 0 1)
+		)
+	)
+	(wire
+		(pts
+			(xy 340.36 100.33) (xy 405.13 100.33)
 		)
 		(stroke
 			(width 2.54)
-			(type solid)
-			(color 194 0 194 1)
-		)
-	)
-	(polyline
-		(pts
-			(xy 433.07 217.17) (xy 433.07 227.33)
-		)
-		(stroke
-			(width 1.27)
-			(type solid)
-			(color 194 0 0 1)
-		)
-	)
-	(polyline
-		(pts
-			(xy 179.07 121.92) (xy 179.07 166.37)
-		)
-		(stroke
-			(width 1.27)
-			(type solid)
-			(color 0 194 0 1)
-		)
-	)
-	(wire
-		(pts
-			(xy 218.44 179.07) (xy 218.44 41.91)
-		)
-		(stroke
-			(width 1.27)
-			(type default)
-			(color 194 0 0 1)
-		)
-	)
-	(wire
-		(pts
-			(xy 340.36 100.33) (xy 405.13 100.33)
+			(type default)
+			(color 255 153 0 1)
+		)
+	)
+	(wire
+		(pts
+			(xy 245.11 101.6) (xy 245.11 49.53)
+		)
+		(stroke
+			(width 1.27)
+			(type default)
+			(color 194 0 0 1)
+		)
+	)
+	(wire
+		(pts
+			(xy 245.11 101.6) (xy 261.62 101.6)
+		)
+		(stroke
+			(width 1.27)
+			(type default)
+			(color 194 0 0 1)
+		)
+	)
+	(wire
+		(pts
+			(xy 384.81 85.09) (xy 384.81 62.23)
 		)
 		(stroke
@@
 	(wire
 		(pts
-			(xy 245.11 101.6) (xy 245.11 49.53)
-		)
-		(stroke
-			(width 1.27)
-			(type default)
-			(color 194 0 0 1)
-		)
-	)
-	(wire
-		(pts
-			(xy 245.11 101.6) (xy 261.62 101.6)
-		)
-		(stroke
-			(width 1.27)
-			(type default)
-			(color 194 0 0 1)
-		)
-	)
-	(wire
-		(pts
-			(xy 384.81 85.09) (xy 384.81 62.23)
-		)
-		(stroke
-			(width 2.54)
-			(type default)
-			(color 255 153 0 1)
+			(xy 680.72 191.77) (xy 711.2 191.77)
+		)
+		(stroke
+			(width 1.27)
+			(type default)
+			(color 50 0 50 1)
 		)
 	)
@@
 		)
 	)
-	(wire
-		(pts
-			(xy 199.39 252.73) (xy 646.43 252.73)
-		)
-		(stroke
-			(width 1.27)
-			(type default)
-			(color 194 0 194 1)
-		)
-	)
 	(polyline
 		(pts
@@
 		)
 	)
+	(wire
+		(pts
+			(xy 109.22 284.48) (xy 109.22 118.11)
+		)
+		(stroke
+			(width 1.27)
+			(type default)
+			(color 50 0 50 1)
+		)
+	)

Commit message: version for piter
Other:
- note added: "Аналоговая цепь 2 х 1,5 кв.мм (например МКЭШ 1,5)"
- note added: "Высокое напряжение постоянное DC 100кв.мм(например, EV-Cable или ППГнг(А)-HF)"
- note added: "Каналы связи с СУ БК 2 х 1,5 кв.мм (например МКЭШ 1,5)"
- note added: "Питание 24В 2 x 4 кв.мм (например, ПВС)"
- note added: "Трехфазный провод с нейтралью 4х10кв.мм (например, КГтп-ХЛ 4х10)"
- note added: "к САУ БК"
- note removed: "Высокое напряжение постоянное DC 100мм2 (например, EV-Cable или ППГнг(А)-HF)"
- note removed: "трехфазный провод с нейтралью 4х10кв.мм (например, КГтп-ХЛ 4х10)"
